File: src/hw/board_files/keypad_usb_hub.kicad_pcb (KiCad board)
At the start: 2 copper layers, 3.4 x 3 mm, 135 parts, among them J1 USB_C_Receptacle_USB2.0_14P, J2 JST S3B-PH-K-S, J3 Conn_ARM_SWD_TagConnect_TC203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, J4 DM3AT-SF-PEJM5, J5 USB_C_Receptacle_USB2.0_14P, J6 Molex 0676433910, J7 Conn_01x04, SW1 RESET, SW10 SW_Push, SW11 SW_Push, SW12 SW_Push, SW13 SW_Push, SW14 SW_Push, SW15 PEC11R-4215K-S0024, SW2 SW_PWR, SW3 SW_Push, SW4 SW_Push, SW5 SW_Push, SW6 SW_Push, SW7 SW_Push, SW8 SW_Push, SW9 SW_Push, U1 USB2514B_Bi, U2 TPS2042D, U3 BQ24074RGT, U4 MDBT50Q-1MV2, U5 XC6220B331MR, U6 W25Q32JVSS, U7 USB2244-AEZG-06, U8 IS31FL3236A-TQ, Y1 24 MHz, Y2 32.768kHz, Y3 24 MHz

Commit message: Working on layout
Parts:
- J1, J7, SW10, SW11, SW12, SW13, SW14, SW15, SW3, SW4, SW5, SW6, SW7, SW8, SW9: moved to B.Cu
- moved SW15 129.6 mm to (164.6, 61.9), turned to 90 degrees
- moved J7 115.5 mm to (186.0, 42.9), turned to -90 degrees
- moved U1 98.5 mm to (34.6, 122.4)
- moved U4 90.8 mm to (144.4, 43.5)
- moved J4 90.1 mm to (129.1, 81.8), turned to -90 degrees
- moved J5 84.8 mm to (125.3, 118.5), turned to -90 degrees
- moved J6 77.1 mm to (134.4, 97.3), turned to -90 degrees
- moved D4 76.0 mm to (23.8, 27.8)
- moved C1 76.0 mm to (26.8, 90.5)
- moved C2 76.0 mm to (26.8, 93.0)
- moved C3 76.0 mm to (26.8, 95.5)
- moved C4 76.0 mm to (26.8, 98.0)
- moved C5 76.0 mm to (26.8, 100.5)
- moved C6 76.0 mm to (26.8, 103.0)
- moved C7 76.0 mm to (27.0, 112.4)
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Other:
- board size 3.4 x 3 mm -> 81.9 x 109.7 mm
